Commit message: Fix a lot problem,rewrote some parts.

File: urdf/two_wheel_cart.urdf (robot description, URDF)
Before this commit: robot two_wheeled_robot, 3 links, 2 joints
Links:
- added link caster_wheel, mass 0.1; collision sphere radius=0.02; visual sphere radius=0.02
- link base_link: mass 5.0 -> 2.0; geometry collision box size=0.4 0.2 0.1; visual box size=0.4 0.2 0.1
- link left_wheel: geometry collision cylinder length=0.03 radius=0.05; visual cylinder length=0.03 radius=0.05
- link right_wheel: geometry collision cylinder length=0.03 radius=0.05; visual cylinder length=0.03 radius=0.05
Joints:
- removed joint left_joint
- removed joint right_joint
- added joint caster_joint: type fixed, parent base_link, child caster_wheel, origin xyz=0.15 0.0 -0.07 rpy=0 0 0
- added joint left_wheel_joint: type continuous, parent base_link, child left_wheel, origin xyz=0.0 0.1 -0.05 rpy=0 0 0, axis 0 1 0
- added joint right_wheel_joint: type continuous, parent base_link, child right_wheel, origin xyz=0.0 -0.1 -0.05 rpy=0 0 0, axis 0 1 0

Commit message: New urdf.

File: urdf/two_wheel_cart.urdf (robot description, URDF)
Before this commit: robot simple_two_wheel_cart, 4 links, 3 joints
Links:
- added link camera_link, mass 0.05; collision box size=0.04 0.05 0.03; visual box size=0.04 0.05 0.03
- added link gimbal_base, mass 0.2; collision cylinder length=0.05 radius=0.03; visual cylinder length=0.05 radius=0.03
- added link gimbal_pitch, mass 0.1; collision box size=0.05 0.05 0.03; visual box size=0.05 0.05 0.03
- added link gimbal_yaw, mass 0.1; collision box size=0.06 0.06 0.04; visual box size=0.06 0.06 0.04
Joints:
- added joint camera_joint: type fixed, parent gimbal_pitch, child camera_link, origin xyz=0.0 0.0 0.03 rpy=0 0 0
- added joint gimbal_base_joint: type fixed, parent base_link, child gimbal_base, origin xyz=0.0 0.0 0.1 rpy=0 0 0
- added joint gimbal_pitch_joint: type revolute, parent gimbal_yaw, child gimbal_pitch, origin xyz=0.0 0.0 0.04 rpy=0 0 0, axis 0 1 0, limit lower=-1.57 upper=1.57 effort=10 velocity=1.0
- added joint gimbal_yaw_joint: type revolute, parent gimbal_base, child gimbal_yaw, origin xyz=0.0 0.0 0.05 rpy=0 0 0, axis 0 0 1, limit lower=-3.14 upper=3.14 effort=10 velocity=1.0
