Commit message: Using ros humble.

File: urdf/mogi_bot_control.xacro (robot description, xacro)
@@ -1,25 +1,25 @@
 <?xml version='1.0'?>
-    <robot name="mogi_bot" xmlns:xacro="http://www.ros.org/wiki/xacro">
-        <xacro:macro name= "mogi_ros2_control">
-            <ros2_control name = "mogi_hardware_interface" type="system">
-                <hardware>
-                    <plugin>gazebo_ros2_control/GazeboSystem</plugin>
-                </hardware>
-                <joint name= "left_wheel_joint">
-                    <command_interface name = "velocity"/>
-                    <state_interface name="velocity"/>
-                    <state_interface name="position"/>
-                </joint>
-                <joint name= "right_wheel_joint">
-                    <command_interface name = "velocity"/>
-                    <state_interface name="velocity"/>
-                    <state_interface name="position"/>
-                </joint>
-            </ros2_control>
-            <gazebo>
-                <plugin filename="libgazebo_ros2_control.so" name="gazebo_ros_control">
-                    <parameters>$(find two_wheel_cart/config/control.yaml)</parameters>
-                </plugin>
-            </gazebo>
-        </xacro:macro>
-    </robot>
+<robot name="mogi_bot" xmlns:xacro="http://www.ros.org/wiki/xacro">
+    <xacro:macro name="mogi_ros2_control">
+        <ros2_control name="mogi_hardware_interface" type="system">
+            <hardware>
+                <plugin>gazebo_ros2_control/GazeboSystem</plugin>
+            </hardware>
+            <joint name="left_wheel_joint">
+                <command_interface name="velocity"/>
+                <state_interface name="position"/>
+                <state_interface name="velocity"/>
+            </joint>
+            <joint name="right_wheel_joint">
+                <command_interface name="velocity"/>
+                <state_interface name="position"/>
+                <state_interface name="velocity"/>
+            </joint>
+        </ros2_control>
+        <gazebo>
+        <plugin filename="libgazebo_ros2_control.so" name="gazebo_ros2_control">
+            <parameters>$(find two_wheeled_cart)/config/controller.yaml</parameters>
+        </plugin>
+        </gazebo>
+    </xacro:macro>
+</robot>
