Commit message: Finish the chassis controller,add camera node.

File: urdf/mogi_bot.urdf2.xacro (robot description, xacro)
@@ -1,5 +1,4 @@
 <?xml version='1.0'?>
-<robot name="mogi_bot" xmlns:xacro="http://www.ros.org/wiki/xacro">
-  <!-- 材料定义 -->
+<robot name="mogi_bot2" xmlns:xacro="http://www.ros.org/wiki/xacro">
   <material name="blue">
     <color rgba="0 0 0.8 1"/>
@@ -17,5 +16,4 @@
     <color rgba="0.8 0.8 0.8 1"/>
   </material>
-  <!-- 参数定义 -->
   <xacro:property name="base_mass" value="15.0" />
   <xacro:property name="wheel_mass" value="5.0" />
@@ -24,5 +22,4 @@
   <xacro:property name="wheel_separation" value="0.3" />
   <xacro:property name="caster_radius" value="0.05" />
-  <!-- 云台参数 -->
   <xacro:property name="gimbal_base_mass" value="0.5" />
   <xacro:property name="gimbal_yaw_mass" value="0.5" />
@@ -31,6 +28,5 @@
   <xacro:property name="barrel_length" value="0.2" />
   <xacro:property name="barrel_radius" value="0.02" />
-  <!-- STEP 1 - Robot footprint -->
-  <link name="base_footprint">
+  <link name="base_footprint2">
     <inertial>
       <mass value="0.001"/>
@@ -38,11 +34,10 @@
     </inertial>
   </link>
-  <!-- STEP 2 - Robot chassis = base_link -->
-  <joint name="base_footprint_joint" type="fixed">
+  <joint name="base_footprint_joint2" type="fixed">
     <origin xyz="0 0 0" rpy="0 0 0" />
-    <parent link="base_footprint"/>
-    <child link="base_link" />
-  </joint>
-  <link name='base_link'>
+    <parent link="base_footprint2"/>
+    <child link="base_link2" />
+  </joint>
+  <link name='base_link2'>
     <inertial>
       <mass value="${base_mass}"/>
@@ -54,5 +49,5 @@
       />
     </inertial>
-    <collision name='collision'>
+    <collision name='collision2'>
       <origin xyz="0 0 0" rpy="0 0 0"/>
       <geometry>
@@ -60,5 +55,5 @@
       </geometry>
     </collision>
-    <visual name='base_link_visual'>
+    <visual name='base_link_visual2'>
       <origin xyz="0 0 0" rpy="0 0 0"/>
       <geometry>
@@ -68,11 +63,10 @@
     </visual>
   </link>
-  <!-- 真正的万向轮结构 -->
-  <link name="caster_wheel_link">
+  <link name="caster_wheel_link2">
     <inertial>
       <mass value="0.1"/>
       <inertia ixx="0.0001" ixy="0.0" ixz="0.0" iyy="0.0001" iyz="0.0" izz="0.0001"/>
     </inertial>
-    <collision name="caster_wheel_collision">
+    <collision name="caster_wheel_collision2">
       <origin xyz="0 0 0" rpy="0 0 0"/>
       <geometry>
@@ -80,5 +74,5 @@
       </geometry>
     </collision>
-    <visual name="caster_wheel_visual">
+    <visual name="caster_wheel_visual2">
       <origin xyz="0 0 0" rpy="0 0 0"/>
       <geometry>
@@ -88,12 +82,11 @@
     </visual>
   </link>
-  <!-- 转向关节 -->
-  <joint name="caster_swivel_joint" type="continuous">
+  <joint name="caster_swivel_joint2" type="continuous">
     <origin xyz="0.25 0 -0.05" rpy="0 0 0"/>
-    <parent link="base_link"/>
-    <child link="caster_swivel_link"/>
+    <parent link="base_link2"/>
+    <child link="caster_swivel_link2"/>
     <axis xyz="0 0 1"/>
   </joint>
-  <link name="caster_swivel_link">
+  <link name="caster_swivel_link2">
     <inertial>
       <mass value="0.05"/>
@@ -101,16 +94,15 @@
     </inertial>
   </link>
-  <!-- 轮子安装关节 -->
-  <joint name="caster_wheel_joint" type="fixed">
+  <joint name="caster_wheel_joint2" type="fixed">
     <origin xyz="0 0 0" rpy="0 0 0"/>
-    <parent link="caster_swivel_link"/>
-    <child link="caster_wheel_link"/>
-  </joint>
-  <link name="caster_wheel_link_2">
+    <parent link="caster_swivel_link2"/>
+    <child link="caster_wheel_link2"/>
+  </joint>
+  <link name="caster_wheel_link_22">
     <inertial>
       <mass value="0.1"/>
       <inertia ixx="0.0001" ixy="0.0" ixz="0.0" iyy="0.0001" iyz="0.0" izz="0.0001"/>
     </inertial>
-    <collision name="caster_wheel_collision_2">
+    <collision name="caster_wheel_collision_22">
       <origin xyz="0 0 0" rpy="0 0 0"/>
       <geometry>
@@ -118,5 +110,5 @@
       </geometry>
     </collision>
-    <visual name="caster_wheel_visual_2">
+    <visual name="caster_wheel_visual_22">
       <origin xyz="0 0 0" rpy="0 0 0"/>
       <geometry>
@@ -126,12 +118,11 @@
     </visual>
   </link>
-  <!-- 转向关节 -->
-  <joint name="caster_swivel_joint_2" type="continuous">
+  <joint name="caster_swivel_joint_22" type="continuous">
     <origin xyz="-0.25 0 -0.05" rpy="0 0 0"/>
-    <parent link="base_link"/>
-    <child link="caster_swivel_link_2"/>
+    <parent link="base_link2"/>
+    <child link="caster_swivel_link_22"/>
     <axis xyz="0 0 1"/>
   </joint>
-  <link name="caster_swivel_link_2">
+  <link name="caster_swivel_link_22">
     <inertial>
       <mass value="0.05"/>
@@ -139,17 +130,15 @@
     </inertial>
   </link>
-  <!-- 轮子安装关节 -->
-  <joint name="caster_wheel_joint_2" type="fixed">
+  <joint name="caster_wheel_joint_22" type="fixed">
     <origin xyz="0 0 0" rpy="0 0 0"/>
-    <parent link="caster_swivel_link_2"/>
-    <child link="caster_wheel_link_2"/>
-  </joint>
-  <!-- STEP 3 - 云台基座 -->
-  <joint name="gimbal_base_joint" type="fixed">
+    <parent link="caster_swivel_link_22"/>
+    <child link="caster_wheel_link_22"/>
+  </joint>
+  <joint name="gimbal_base_joint2" type="fixed">
     <origin xyz="0.1 0 0.05" rpy="0 0 0" />
-    <parent link="base_link"/>
-    <child link="gimbal_base" />
-  </joint>
-  <link name='gimbal_base'>
+    <parent link="base_link2"/>
+    <child link="gimbal_base2" />
+  </joint>
+  <link name='gimbal_base2'>
     <inertial>
       <mass value="${gimbal_base_mass}"/>
@@ -161,5 +150,5 @@
       />
     </inertial>
-    <collision name='gimbal_base_collision'>
+    <collision name='gimbal_base_collision2'>
       <origin xyz="0 0 0.02" rpy="0 0 0"/>
       <geometry>
@@ -167,5 +156,5 @@
       </geometry>
     </collision>
-    <visual name='gimbal_base_visual'>
+    <visual name='gimbal_base_visual2'>
       <origin xyz="0 0 0.02" rpy="0 0 0"/>
       <geometry>
@@ -175,13 +164,12 @@
     </visual>
   </link>
-  <!-- STEP 4 - 云台偏航关节 (Yaw) -->
-  <joint name="gimbal_yaw_joint" type="revolute">
+  <joint name="gimbal_yaw_joint2" type="revolute">
     <origin xyz="0 0 0.04" rpy="0 0 0" />
-    <parent link="gimbal_base"/>
-    <child link="gimbal_yaw" />
+    <parent link="gimbal_base2"/>
+    <child link="gimbal_yaw2" />
     <axis xyz="0 0 1" />
     <limit lower="-3.14" upper="3.14" effort="10" velocity="2.0"/>
   </joint>
-  <link name='gimbal_yaw'>
+  <link name='gimbal_yaw2'>
     <inertial>
       <mass value="${gimbal_yaw_mass}"/>
@@ -193,5 +181,5 @@
       />
     </inertial>
-    <collision name='gimbal_yaw_collision'>
+    <collision name='gimbal_yaw_collision2'>
       <origin xyz="0 0 0.02" rpy="0 0 0"/>
       <geometry>
@@ -199,5 +187,5 @@
       </geometry>
     </collision>
-    <visual name='gimbal_yaw_visual'>
+    <visual name='gimbal_yaw_visual2'>
       <origin xyz="0 0 0.02" rpy="0 0 0"/>
       <geometry>
@@ -207,11 +195,10 @@
     </visual>
   </link>
-  <!-- STEP 5 - 枪管连接 -->
-  <joint name="barrel_joint" type="fixed">
+  <joint name="barrel_joint2" type="fixed">
     <origin xyz="0 0 0.04" rpy="0 0 0" />
-    <parent link="gimbal_yaw"/>
-    <child link="barrel_link" />
-  </joint>
-  <link name='barrel_link'>
+    <parent link="gimbal_yaw2"/>
+    <child link="barrel_link2" />
+  </joint>
+  <link name='barrel_link2'>
     <inertial>
       <mass value="${barrel_mass}"/>
@@ -223,5 +210,5 @@
       />
     </inertial>
-    <collision name='barrel_collision'>
+    <collision name='barrel_collision2'>
       <origin xyz="${barrel_length/2} 0 0" rpy="1.57 0 1.57"/>
       <geometry>
@@ -229,5 +216,5 @@
       </geometry>
     </collision>
-    <visual name='barrel_visual'>
+    <visual name='barrel_visual2'>
       <origin xyz="${barrel_length/2} 0 0" rpy="1.57 0 1.57"/>
       <geometry>
@@ -237,11 +224,10 @@
     </visual>
   </link>
-  <!-- STEP 6 - 相机安装在枪管末端 -->
-  <joint name="camera_joint" type="fixed">
+  <joint name="camera_joint2" type="fixed">
     <origin xyz="${barrel_length} 0 0" rpy="0 0 0" />
-    <parent link="barrel_link"/>
-    <child link="camera_link" />
-  </joint>
-  <link name='camera_link'>
+    <parent link="barrel_link2"/>
+    <child link="camera_link2" />
+  </joint>
+  <link name='camera_link2'>
     <inertial>
       <mass value="${camera_mass}"/>
@@ -253,5 +239,5 @@
       />
     </inertial>
-    <visual name='camera_visual'>
+    <visual name='camera_visual2'>
       <origin xyz="0 0 0" rpy="0 1.5708 1.5708"/>
       <geometry>
@@ -260,5 +246,5 @@
       <material name="black"/>
     </visual>
-    <visual name='camera_lens_visual'>
+    <visual name='camera_lens_visual2'>
       <origin xyz="0.02 0 0" rpy="0 1.5708 1.5708"/>
       <geometry>
@@ -267,5 +253,5 @@
       <material name="white"/>
     </visual>
-    <collision name='camera_collision'>
+    <collision name='camera_collision2'>
       <origin xyz="0 0 0" rpy="0 1.5708 1.5708"/>
       <geometry>
@@ -273,8 +259,7 @@
       </geometry>
     </collision>
-    <!-- 相机传感器 -->
-    <sensor name="camera_sensor" type="camera">
+    <sensor name="camera_sensor2" type="camera">
       <pose>0.02 0 0 0 -1.5708 1.5708</pose>
-      <camera name="camera">
+      <camera name="camera2">
         <horizontal_fov>1.0472</horizontal_fov>
         <image>
@@ -297,14 +282,13 @@
     </sensor>
   </link>
-  <!-- STEP 7 - 左轮 -->
-  <joint type="continuous" name="left_wheel_joint">
+  <joint type="continuous" name="left_wheel_joint2">
     <origin xyz="0 0.125 0" rpy="0 0 0"/>
-    <child link="left_wheel"/>
-    <parent link="base_link"/>
+    <child link="left_wheel2"/>
+    <parent link="base_link2"/>
     <axis xyz="0 1 0" rpy="0 0 0"/>
     <limit effort="100" velocity="10"/>
     <dynamics damping="1.0" friction="1.0"/>
   </joint>
-  <link name='left_wheel'>
+  <link name='left_wheel2'>
     <inertial>
       <mass value="${wheel_mass}"/>
@@ -316,5 +300,5 @@
       />
     </inertial>
-    <collision name="left_wheel_collision">
+    <collision name="left_wheel_collision2">
       <origin xyz="0 0 0" rpy="0 1.5707 1.5707"/>
       <geometry>
@@ -322,5 +306,5 @@
       </geometry>
     </collision>
-    <visual name='left_wheel_visual'>
+    <visual name='left_wheel_visual2'>
       <origin xyz="0 0 0" rpy="0 1.5707 1.5707"/>
       <geometry>
@@ -330,14 +314,13 @@
     </visual>
   </link>
-  <!-- STEP 8 - 右轮 -->
-  <joint type="continuous" name="right_wheel_joint">
+  <joint type="continuous" name="right_wheel_joint2">
     <origin xyz="0 -0.125 0" rpy="0 0 0"/>
-    <child link="right_wheel"/>
-    <parent link="base_link"/>
+    <child link="right_wheel2"/>
+    <parent link="base_link2"/>
     <axis xyz="0 1 0" rpy="0 0 0"/>
     <limit effort="100" velocity="10"/>
     <dynamics damping="1.0" friction="1.0"/>
   </joint>
-  <link name='right_wheel'>
+  <link name='right_wheel2'>
     <inertial>
       <mass value="${wheel_mass}"/>
@@ -349,5 +332,5 @@
       />
     </inertial>
-    <collision name="right_wheel_collision">
+    <collision name="right_wheel_collision2">
       <origin xyz="0 0 0" rpy="0 1.5707 1.5707"/>
       <geometry>
@@ -355,5 +338,5 @@
       </geometry>
     </collision>
-    <visual name='right_wheel_visual'>
+    <visual name='right_wheel_visual2'>
       <origin xyz="0 0 0" rpy="0 1.5707 1.5707"/>
       <geometry>
@@ -363,15 +346,13 @@
     </visual>
   </link>
-  <!-- Gazebo 插件配置 -->
   <gazebo>
-    <plugin name="gazebo_ros2_control" filename="libgazebo_ros2_control.so">
+    <plugin name="gazebo_ros2_control2" filename="libgazebo_ros2_control.so">
       <parameters>$(find two_wheeled_cart)/config/controller.yaml</parameters>
     </plugin>
   </gazebo>
-  <!-- 相机 Gazebo 插件 -->
-  <gazebo reference="camera_link">
-    <sensor type="camera" name="camera1">
+  <gazebo reference="camera_link2">
+    <sensor type="camera" name="camera12">
       <update_rate>30.0</update_rate>
-      <camera name="head">
+      <camera name="head2">
         <horizontal_fov>1.0472</horizontal_fov>
         <image>
@@ -385,34 +366,31 @@
         </clip>
       </camera>
-      <plugin name="camera_controller" filename="libgazebo_ros_camera.so">
+      <plugin name="camera_controller2" filename="libgazebo_ros_camera.so">
         <ros>
-          <namespace>/mogi_bot</namespace>
+          <namespace>/mogi_bot2</namespace>
           <remapping>image_raw:=camera/image_raw</remapping>
           <remapping>camera_info:=camera/camera_info</remapping>
         </ros>
-        <camera_name>camera</camera_name>
-        <frame_name>camera_link</frame_name>
+        <camera_name>camera2</camera_name>
+        <frame_name>camera_link2</frame_name>
         <hack_baseline>0.07</hack_baseline>
       </plugin>
     </sensor>
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