Commit message: Fof four wheel car.

File: urdf/mogi_bot.urdf.xacro (robot description, xacro)
@@ -8,28 +8,15 @@
     <color rgba="0 0 0 1"/>
   </material>
-  <material name="white">
-    <color rgba="1 1 1 1"/>
-  </material>
   <material name="gray">
     <color rgba="0.5 0.5 0.5 1"/>
   </material>
-  <material name="silver">
-    <color rgba="0.8 0.8 0.8 1"/>
-  </material>
-  <!-- 参数定义 -->
+  <!-- 核心参数定义（四轮小车适配） -->
   <xacro:property name="base_mass" value="15.0" />
   <xacro:property name="wheel_mass" value="5.0" />
   <xacro:property name="wheel_radius" value="0.1" />
   <xacro:property name="wheel_length" value="0.05" />
-  <xacro:property name="wheel_separation" value="0.3" />
-  <xacro:property name="caster_radius" value="0.05" />
-  <!-- 云台参数 -->
-  <xacro:property name="gimbal_base_mass" value="0.5" />
-  <xacro:property name="gimbal_yaw_mass" value="0.5" />
-  <xacro:property name="barrel_mass" value="0.3" />
-  <xacro:property name="camera_mass" value="0.3" />
-  <xacro:property name="barrel_length" value="0.2" />
-  <xacro:property name="barrel_radius" value="0.02" />
-  <!-- STEP 1 - Robot footprint -->
+  <xacro:property name="wheel_separation" value="0.3" /> <!-- 左右轮间距 -->
+  <xacro:property name="wheelbase" value="0.4" />        <!-- 前后轮间距 -->
+  <!-- 1. 基准坐标系 -->
   <link name="base_footprint">
     <inertial>
@@ -38,5 +25,5 @@
     </inertial>
   </link>
-  <!-- STEP 2 - Robot chassis = base_link -->
+  <!-- 2. 车身底座（base_link） -->
   <joint name="base_footprint_joint" type="fixed">
     <origin xyz="0 0 0" rpy="0 0 0" />
@@ -68,358 +55,168 @@
     </visual>
   </link>
-  <!-- 真正的万向轮结构 -->
-  <link name="caster_wheel_link">
-    <inertial>
-      <mass value="0.1"/>
-      <inertia ixx="0.0001" ixy="0.0" ixz="0.0" iyy="0.0001" iyz="0.0" izz="0.0001"/>
-    </inertial>
-    <collision name="caster_wheel_collision">
-      <origin xyz="0 0 0" rpy="0 0 0"/>
-      <geometry>
-        <sphere radius="0.05"/>
-      </geometry>
-    </collision>
-    <visual name="caster_wheel_visual">
-      <origin xyz="0 0 0" rpy="0 0 0"/>
-      <geometry>
-        <sphere radius="0.05"/>
-      </geometry>
-      <material name="black"/>
-    </visual>
-  </link>
-  <!-- 转向关节 -->
-  <joint name="caster_swivel_joint" type="continuous">
-    <origin xyz="0.25 0 -0.05" rpy="0 0 0"/>
-    <parent link="base_link"/>
-    <child link="caster_swivel_link"/>
-    <axis xyz="0 0 1"/>
-  </joint>
-  <link name="caster_swivel_link">
-    <inertial>
-      <mass value="0.05"/>
-      <inertia ixx="0.00001" ixy="0.0" ixz="0.0" iyy="0.00001" iyz="0.0" izz="0.00001"/>
-    </inertial>
-  </link>
-  <!-- 轮子安装关节 -->
-  <joint name="caster_wheel_joint" type="fixed">
-    <origin xyz="0 0 0" rpy="0 0 0"/>
-    <parent link="caster_swivel_link"/>
-    <child link="caster_wheel_link"/>
-  </joint>
-  <link name="caster_wheel_link_2">
-    <inertial>
-      <mass value="0.1"/>
-      <inertia ixx="0.0001" ixy="0.0" ixz="0.0" iyy="0.0001" iyz="0.0" izz="0.0001"/>
-    </inertial>
-    <collision name="caster_wheel_collision_2">
-      <origin xyz="0 0 0" rpy="0 0 0"/>
-      <geometry>
-        <sphere radius="0.05"/>
-      </geometry>
-    </collision>
-    <visual name="caster_wheel_visual_2">
-      <origin xyz="0 0 0" rpy="0 0 0"/>
-      <geometry>
-        <sphere radius="0.05"/>
-      </geometry>
-      <material name="black"/>
-    </visual>
-  </link>
-  <!-- 转向关节 -->
-  <joint name="caster_swivel_joint_2" type="continuous">
-    <origin xyz="-0.25 0 -0.05" rpy="0 0 0"/>
-    <parent link="base_link"/>
-    <child link="caster_swivel_link_2"/>
-    <axis xyz="0 0 1"/>
-  </joint>
-  <link name="caster_swivel_link_2">
-    <inertial>
-      <mass value="0.05"/>
-      <inertia ixx="0.00001" ixy="0.0" ixz="0.0" iyy="0.00001" iyz="0.0" izz="0.00001"/>
-    </inertial>
-  </link>
-  <!-- 轮子安装关节 -->
-  <joint name="caster_wheel_joint_2" type="fixed">
-    <origin xyz="0 0 0" rpy="0 0 0"/>
-    <parent link="caster_swivel_link_2"/>
-    <child link="caster_wheel_link_2"/>
-  </joint>
-  <!-- STEP 3 - 云台基座 -->
-  <joint name="gimbal_base_joint" type="fixed">
-    <origin xyz="0.1 0 0.05" rpy="0 0 0" />
-    <parent link="base_link"/>
-    <child link="gimbal_base" />
-  </joint>
-  <link name='gimbal_base'>
-    <inertial>
-      <mass value="${gimbal_base_mass}"/>
-      <origin xyz="0 0 0.02" rpy="0 0 0"/>
-      <inertia
-          ixx="0.001" ixy="0" ixz="0"
-          iyy="0.001" iyz="0"
-          izz="0.001"
-      />
-    </inertial>
-    <collision name='gimbal_base_collision'>
-      <origin xyz="0 0 0.02" rpy="0 0 0"/>
-      <geometry>
-        <cylinder radius="0.04" length="0.04"/>
-      </geometry>
-    </collision>
-    <visual name='gimbal_base_visual'>
-      <origin xyz="0 0 0.02" rpy="0 0 0"/>
-      <geometry>
-        <cylinder radius="0.04" length="0.04"/>
-      </geometry>
-      <material name="silver"/>
-    </visual>
-  </link>
-  <!-- STEP 4 - 云台偏航关节 (Yaw) -->
-  <joint name="gimbal_yaw_joint" type="revolute">
-    <origin xyz="0 0 0.04" rpy="0 0 0" />
-    <parent link="gimbal_base"/>
-    <child link="gimbal_yaw" />
-    <axis xyz="0 0 1" />
-    <limit lower="-3.14" upper="3.14" effort="10" velocity="2.0"/>
-  </joint>
-  <link name='gimbal_yaw'>
-    <inertial>
-      <mass value="${gimbal_yaw_mass}"/>
-      <origin xyz="0 0 0.02" rpy="0 0 0"/>
-      <inertia
-          ixx="0.0005" ixy="0" ixz="0"
-          iyy="0.0005" iyz="0"
-          izz="0.0005"
-      />
-    </inertial>
-    <collision name='gimbal_yaw_collision'>
-      <origin xyz="0 0 0.02" rpy="0 0 0"/>
-      <geometry>
-        <box size="0.08 0.08 0.04"/>
-      </geometry>
-    </collision>
-    <visual name='gimbal_yaw_visual'>
-      <origin xyz="0 0 0.02" rpy="0 0 0"/>
-      <geometry>
-        <box size="0.08 0.08 0.04"/>
-      </geometry>
-      <material name="gray"/>
-    </visual>
-  </link>
-  <!-- STEP 5 - 枪管连接 -->
-  <joint name="barrel_joint" type="fixed">
-    <origin xyz="0 0 0.04" rpy="0 0 0" />
-    <parent link="gimbal_yaw"/>
-    <child link="barrel_link" />
-  </joint>
-  <link name='barrel_link'>
-    <inertial>
-      <mass value="${barrel_mass}"/>
-      <origin xyz="${barrel_length/2} 0 0" rpy="0 0 0"/>
-      <inertia
-          ixx="0.0003" ixy="0" ixz="0"
-          iyy="0.0003" iyz="0"
-          izz="0.0003"
-      />
-    </inertial>
-    <collision name='barrel_collision'>
-      <origin xyz="${barrel_length/2} 0 0" rpy="1.57 0 1.57"/>
-      <geometry>
-        <cylinder radius="${barrel_radius}" length="${barrel_length}"/>
-      </geometry>
-    </collision>
-    <visual name='barrel_visual'>
-      <origin xyz="${barrel_length/2} 0 0" rpy="1.57 0 1.57"/>
-      <geometry>
-        <cylinder radius="${barrel_radius}" length="${barrel_length}"/>
-      </geometry>
-      <material name="black"/>
-    </visual>
-  </link>
-  <!-- STEP 6 - 相机安装在枪管末端 -->
-  <joint name="camera_joint" type="fixed">
-    <origin xyz="${barrel_length} 0 0" rpy="0 0 0" />
-    <parent link="barrel_link"/>
-    <child link="camera_link" />
-  </joint>
-  <link name='camera_link'>
-    <inertial>
-      <mass value="${camera_mass}"/>
-      <origin xyz="0 0 0" rpy="0 0 0"/>
-      <inertia
-          ixx="0.0001" ixy="0" ixz="0"
-          iyy="0.0001" iyz="0"
-          izz="0.0001"
-      />
-    </inertial>
-    <visual name='camera_visual'>
-      <origin xyz="0 0 0" rpy="0 1.5708 1.5708"/>
-      <geometry>
-        <cylinder radius="0.015" length="0.04"/>
-      </geometry>
-      <material name="black"/>
-    </visual>
-    <visual name='camera_lens_visual'>
-      <origin xyz="0.02 0 0" rpy="0 1.5708 1.5708"/>
-      <geometry>
-        <cylinder radius="0.008" length="0.005"/>
-      </geometry>
-      <material name="white"/>
-    </visual>
-    <collision name='camera_collision'>
-      <origin xyz="0 0 0" rpy="0 1.5708 1.5708"/>
-      <geometry>
-        <cylinder radius="0.015" length="0.04"/>
-      </geometry>
-    </collision>
-    <!-- 相机传感器 -->
-    <sensor name="camera_sensor" type="camera">
-      <pose>0.02 0 0 0 -1.5708 1.5708</pose>
-      <camera name="camera">
-        <horizontal_fov>1.0472</horizontal_fov>
-        <image>
-          <width>640</width>
-          <height>480</height>
-          <format>R8G8B8</format>
-        </image>
-        <clip>
-          <near>0.05</near>
-          <far>100</far>
-        </clip>
-        <noise>
-          <type>gaussian</type>
-          <mean>0.0</mean>
-          <stddev>0.007</stddev>
-        </noise>
-      </camera>
-      <always_on>1</always_on>
-      <update_rate>30</update_rate>
-    </sensor>
-  </link>
-  <!-- STEP 7 - 左轮 -->
-  <joint type="continuous" name="left_wheel_joint">
-    <origin xyz="0 0.125 0" rpy="0 0 0"/>
-    <child link="left_wheel"/>
-    <parent link="base_link"/>
-    <axis xyz="0 1 0" rpy="0 0 0"/>
-    <limit effort="100" velocity="10"/>
-    <dynamics damping="1.0" friction="1.0"/>
-  </joint>
-  <link name='left_wheel'>
-    <inertial>
-      <mass value="${wheel_mass}"/>
-      <origin xyz="0 0 0" rpy="0 1.5707 1.5707"/>
-      <inertia
-          ixx="0.014" ixy="0" ixz="0"
-          iyy="0.014" iyz="0"
-          izz="0.025"
-      />
-    </inertial>
-    <collision name="left_wheel_collision">
-      <origin xyz="0 0 0" rpy="0 1.5707 1.5707"/>
-      <geometry>
-        <cylinder radius="${wheel_radius}" length="${wheel_length}"/>
-      </geometry>
-    </collision>
-    <visual name='left_wheel_visual'>
-      <origin xyz="0 0 0" rpy="0 1.5707 1.5707"/>
-      <geometry>
-        <cylinder radius="${wheel_radius}" length="${wheel_length}"/>
-      </geometry>
-      <material name="black"/>
-    </visual>
-  </link>
-  <!-- STEP 8 - 右轮 -->
-  <joint type="continuous" name="right_wheel_joint">
-    <origin xyz="0 -0.125 0" rpy="0 0 0"/>
-    <child link="right_wheel"/>
-    <parent link="base_link"/>
-    <axis xyz="0 1 0" rpy="0 0 0"/>
-    <limit effort="100" velocity="10"/>
-    <dynamics damping="1.0" friction="1.0"/>
-  </joint>
-  <link name='right_wheel'>
-    <inertial>
-      <mass value="${wheel_mass}"/>
-      <origin xyz="0 0 0" rpy="0 1.5707 1.5707"/>
-      <inertia
-          ixx="0.014" ixy="0" ixz="0"
-          iyy="0.014" iyz="0"
-          izz="0.025"
-      />
-    </inertial>
-    <collision name="right_wheel_collision">
-      <origin xyz="0 0 0" rpy="0 1.5707 1.5707"/>
-      <geometry>
-        <cylinder radius="${wheel_radius}" length="${wheel_length}"/>
-      </geometry>
-    </collision>
-    <visual name='right_wheel_visual'>
-      <origin xyz="0 0 0" rpy="0 1.5707 1.5707"/>
-      <geometry>
-        <cylinder radius="${wheel_radius}" length="${wheel_length}"/>
-      </geometry>
-      <material name="black"/>
-    </visual>
-  </link>
-  <!-- Gazebo 插件配置 -->
+  <!-- 3. 四轮驱动结构 -->
+  <!-- 前轮（左） -->
+  <joint type="continuous" name="front_left_wheel_joint">
+    <origin xyz="${wheelbase/2} ${wheel_separation/2} 0" rpy="0 0 0"/>
+    <child link="front_left_wheel"/>
+    <parent link="base_link"/>
+    <axis xyz="0 1 0"/>
+    <limit effort="100" velocity="10"/>
+    <dynamics damping="1.0" friction="1.0"/>
+  </joint>
+  <link name='front_left_wheel'>
+    <inertial>
+      <mass value="${wheel_mass}"/>
+      <origin xyz="0 0 0" rpy="0 1.5707 1.5707"/>
+      <inertia
+          ixx="0.014" ixy="0" ixz="0"
+          iyy="0.014" iyz="0"
+          izz="0.025"
+      />
+    </inertial>
+    <collision name="front_left_wheel_collision">
+      <origin xyz="0 0 0" rpy="0 1.5707 1.5707"/>
+      <geometry>
+        <cylinder radius="${wheel_radius}" length="${wheel_length}"/>
+      </geometry>
+    </collision>
+    <visual name='front_left_wheel_visual'>
+      <origin xyz="0 0 0" rpy="0 1.5707 1.5707"/>
+      <geometry>
+        <cylinder radius="${wheel_radius}" length="${wheel_length}"/>
+      </geometry>
+      <material name="black"/>
+    </visual>
+  </link>
+  <!-- 前轮（右） -->
+  <joint type="continuous" name="front_right_wheel_joint">
+    <origin xyz="${wheelbase/2} -${wheel_separation/2} 0" rpy="0 0 0"/>
+    <child link="front_right_wheel"/>
+    <parent link="base_link"/>
+    <axis xyz="0 1 0"/>
+    <limit effort="100" velocity="10"/>
+    <dynamics damping="1.0" friction="1.0"/>
+  </joint>
+  <link name='front_right_wheel'>
+    <inertial>
+      <mass value="${wheel_mass}"/>
+      <origin xyz="0 0 0" rpy="0 1.5707 1.5707"/>
+      <inertia
+          ixx="0.014" ixy="0" ixz="0"
+          iyy="0.014" iyz="0"
+          izz="0.025"
+      />
+    </inertial>
+    <collision name="front_right_wheel_collision">
+      <origin xyz="0 0 0" rpy="0 1.5707 1.5707"/>
+      <geometry>
+        <cylinder radius="${wheel_radius}" length="${wheel_length}"/>
+      </geometry>
+    </collision>
+    <visual name='front_right_wheel_visual'>
+      <origin xyz="0 0 0" rpy="0 1.5707 1.5707"/>
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
Commit message: Finish the traject.

File: urdf/mogi_bot.urdf.xacro (robot description, xacro)
@@ -18,5 +18,16 @@
   <xacro:property name="wheel_separation" value="0.3" /> <!-- 左右轮间距 -->
   <xacro:property name="wheelbase" value="0.4" />        <!-- 前后轮间距 -->
-  <!-- 1. 基准坐标系 -->
+  <link name="odom">
+      <inertial>
+        <mass value="0.001"/>
+        <inertia ixx="0.001" ixy="0.0" ixz="0.0" iyy="0.001" iyz="0.0" izz="0.001"/>
+      </inertial>
+    </link>
+    <!-- 新增：odom 到 base_footprint 的固定关节（里程计坐标系关联） -->
+    <joint name="odom_joint" type="fixed">
+      <origin xyz="0 0 0" rpy="0 0 0" />
+      <parent link="odom"/>
+      <child link="base_footprint"/>
+    </joint>
   <link name="base_footprint">
     <inertial>
